File: src/Mix necessary function.brd (EAGLE design)
At the start: 53 x 42 mm, 15 parts, among them CON1 XT90PW-M, SW1 02-JST, SW2 02-JST

Commit message: servo2
Parts:
- added LED_SW: SS-12SDP2, SS-12SDP2:SS-12SDP2
- moved AZUSA 2.00 mm to (44.4, 21.4)
Connections:
- new net BLUE: LED.1, LED_SW.L
- new net RED: LED.2, LED_SW.R
- net GND: now also LED_SW.C; no longer LED.1, LED.3
Routing:
- net RED: track 0.00 -> 18.1 mm
- net BLUE: track 0.00 -> 13.2 mm
- net VCC: track 11.4 -> 9.43 mm
Other:
- outline, holes or cut-outs redrawn
Changed lines of the file:
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@@
 <drawing>
 <settings>
-<setting alwaysvectorfont="yes"/>
+<setting alwaysvectorfont="no"/>
 <setting verticaltext="up"/>
 </settings>
@@
 <board>
 <plain>
-<wire x1="0" y1="0" x2="53" y2="0" width="0" layer="20"/>
-<wire x1="53" y1="0" x2="53" y2="42" width="0" layer="20"/>
-<wire x1="53" y1="42" x2="0" y2="42" width="0" layer="20"/>
-<wire x1="0" y1="42" x2="0" y2="0" width="0" layer="20"/>
+<wire x1="0" y1="39" x2="0" y2="3" width="0" layer="20"/>
+<wire x1="0" y1="3" x2="3" y2="0" width="0" layer="20" curve="90"/>
+<wire x1="3" y1="0" x2="50" y2="0" width="0" layer="20"/>
+<wire x1="50" y1="0" x2="53" y2="3" width="0" layer="20" curve="90"/>
+<wire x1="53" y1="3" x2="53" y2="39" width="0" layer="20"/>
+<wire x1="53" y1="39" x2="50" y2="42" width="0" layer="20" curve="90"/>
+<wire x1="50" y1="42" x2="3" y2="42" width="0" layer="20"/>
+<wire x1="3" y1="42" x2="0" y2="39" width="0" layer="20" curve="90"/>
 </plain>
 <attributes>
@@
 <attribute name="VALUE" x="39.29" y="0.62" size="1.27" layer="27"/>
 </element>
-<element name="AZUSA" library="con-jst-xh (1)" package="B2B-XH" value="02-JST" x="44.42" y="19.43" smashed="yes">
-<attribute name="NAME" x="41.499" y="23.113" size="1.27" layer="25"/>
-<attribute name="VALUE" x="43.15" y="15.62" size="1.27" layer="27"/>
+<element name="AZUSA" library="con-jst-xh (1)" package="B2B-XH" value="02-JST" x="44.42" y="21.43" smashed="yes">
+<attribute name="NAME" x="41.499" y="25.113" size="1.27" layer="25"/>
+<attribute name="VALUE" x="43.15" y="17.62" size="1.27" layer="27"/>
 </element>
 <element name="SW1" library="con-jst-xh (1)" package="B2B-XH" value="02-JST" x="44.42" y="30.86" smashed="yes">
@@
 <attribute name="NAME" x="33.9905" y="10.8705" size="0.5" layer="25" rot="R270"/>
 <attribute name="VALUE" x="35.0405" y="10.8705" size="0.5" layer="27" rot="R270"/>
+</element>
+<element name="LED_SW" library="SS-12SDP2" package="SS-12SDP2" value="SS-12SDP2" x="44" y="13" smashed="yes">
+<attribute name="VALUE" x="39.047" y="15.286" size="0.7" layer="27"/>
 </element>
 </elements>
@@
 <contactref element="U$17" pad="GND"/>
 <contactref element="C5" pad="2"/>
-<contactref element="LED" pad="3"/>
-<contactref element="LED" pad="1"/>
 <contactref element="AZUSA_CON" pad="1"/>
 <contactref element="SERVO" pad="1"/>
@@
 <vertex x="-1" y="45"/>
 </polygon>
-<wire x1="34.778" y1="22.001" x2="35.53" y2="30.86" width="0" layer="19" extent="1-1"/>
-<wire x1="33.587" y1="22.001" x2="34.778" y2="22.001" width="0" layer="19" extent="1-1"/>
-<wire x1="31" y1="20" x2="33.587" y2="22.001" width="0" layer="19" extent="1-1"/>
-<wire x1="27.068" y1="16.832" x2="31" y2="20" width="0" layer="19" extent="1-1"/>
-<wire x1="27.068" y1="12.871" x2="27.068" y2="16.832" width="0" layer="19" extent="1-1"/>
-<wire x1="33.587" y1="9.233" x2="27.068" y2="12.871" width="0" layer="19" extent="1-1"/>
-<wire x1="34.778" y1="9.233" x2="33.587" y2="9.233" width="0" layer="19" extent="1-1"/>
-<wire x1="28" y1="5" x2="33.587" y2="9.233" width="0" layer="19" extent="1-1"/>
-<wire x1="41.83" y1="4.43" x2="34.778" y2="9.233" width="0" layer="19" extent="1-1"/>
-<wire x1="46.91" y1="4.43" x2="41.83" y2="4.43" width="0" layer="19" extent="1-1"/>
-<wire x1="19.27" y1="5" x2="28" y2="5" width="0" layer="19" extent="1-1"/>
-<wire x1="9.54" y1="5" x2="19.27" y2="5" width="0" layer="19" extent="1-1"/>
-<wire x1="45.69" y1="19.43" x2="34.778" y2="22.001" width="0" layer="19" extent="1-1"/>
-<wire x1="21" y1="30.45" x2="31" y2="20" width="0" layer="19" extent="1-1"/>
+<contactref element="LED_SW" pad="C"/>
 </signal>
 <signal name="VCC">
 <contactref element="SW1" pad="2"/>
 <contactref element="AZUSA" pad="2"/>
-<wire x1="43.15" y1="19.43" x2="43.15" y2="30.86" width="1.016" layer="1"/>
+<wire x1="43.15" y1="21.43" x2="43.15" y2="30.86" width="1.016" layer="1"/>
 </signal>
 <signal name="EM">
 <contactref element="SW1" pad="1"/>
 <contactref element="SW2" pad="2"/>
-<wire x1="32.99" y1="30.86" x2="33.08805625" y2="30.86" width="1.016" layer="1"/>
-<wire x1="33.08805625" y1="30.86" x2="34.50245625" y2="32.2744" width="1.016" layer="1"/>
+<wire x1="34.50245625" y1="32.5284" x2="32.99" y2="31.01594375" width="1.016" layer="1"/>
+<wire x1="32.99" y1="30.86" x2="32.99" y2="31.01594375" width="1.016" layer="1"/>
 <wire x1="45.69" y1="30.86" x2="45.69" y2="31.32026875" width="1.016" layer="1"/>
-<wire x1="45.69" y1="31.32026875" x2="44.73586875" y2="32.2744" width="1.016" layer="1"/>
-<wire x1="34.50245625" y1="32.2744" x2="44.73586875" y2="32.2744" width="1.016" layer="1"/>
+<wire x1="45.69" y1="31.32026875" x2="44.48186875" y2="32.5284" width="1.016" layer="1"/>
+<wire x1="34.50245625" y1="32.5284" x2="44.48186875" y2="32.5284" width="1.016" layer="1"/>
 </signal>
 <signal name="PVCC">
@@
 <wire x1="26.479" y1="13.521" x2="27.068" y2="13.521" width="0.5" layer="1"/>
 <wire x1="27.068" y1="13.521" x2="27.479" y2="13.521" width="0.5" layer="1"/>
-<wire x1="33.35" y1="3.48091875" x2="33.35" y2="2.7" width="0.5" layer="1"/>
-<wire x1="31.5706" y1="9.4294" x2="31.5706" y2="5.26031875" width="0.5" layer="1"/>
-<wire x1="31.5706" y1="5.26031875" x2="33.35" y2="3.48091875" width="0.5" layer="1"/>
+<wire x1="33.35" y1="4.24291875" x2="33.35" y2="2.7" width="0.5" layer="1"/>
+<wire x1="31.5706" y1="9.4294" x2="31.5706" y2="6.02231875" width="0.5" layer="1"/>
+<wire x1="31.5706" y1="6.02231875" x2="33.35" y2="4.24291875" width="0.5" layer="1"/>
 <wire x1="27.479" y1="13.521" x2="31.5706" y2="9.4294" width="0.5" layer="1"/>
 </signal>
@@
 <wire x1="33.587" y1="22.651" x2="34.778" y2="22.651" width="0.5" layer="1"/>
 </signal>
+<signal name="RED">
+<contactref element="LED" pad="2"/>
+<contactref element="LED_SW" pad="R"/>
+<wire x1="46.54" y1="13" x2="49" y2="10.54" width="0.1524" layer="1"/>
+<wire x1="49" y1="10.54" x2="49" y2="3" width="0.1524" layer="1"/>
+<wire x1="49" y1="3" x2="48" y2="2" width="0.1524" layer="1"/>
+<wire x1="48" y1="2" x2="45" y2="2" width="0.1524" layer="1"/>
+<wire x1="45" y1="2" x2="44.37" y2="2.63" width="0.1524" layer="1"/>
+<wire x1="44.37" y1="2.63" x2="44.37" y2="4.43" width="0.1524" layer="1"/>
+</signal>
+<signal name="BLUE">
+<contactref element="LED" pad="1"/>
+<contactref element="LED_SW" pad="L"/>
+<wire x1="41.46" y1="13" x2="41.46" y2="7.54" width="0.1524" layer="1"/>
+<wire x1="41.46" y1="7.54" x2="42" y2="7" width="0.1524" layer="1"/>
+<wire x1="42" y1="7" x2="46" y2="7" width="0.1524" layer="1"/>
+<wire x1="46" y1="7" x2="46.91" y2="6.09" width="0.1524" layer="1"/>
+<wire x1="46.91" y1="6.09" x2="46.91" y2="4.43" width="0.1524" layer="1"/>
+</signal>
 </signals>

Commit message: necefunc fix
Parts:
- removed AZUSA_CON: 02-JST, con-jst-xh (1):B2B-XH
- removed SERVO: (no value), con-jst-xh (1):B3B-XH
- added AZUSA_CON1, AZUSA_CON2: 02-JST, con-jst-xh (1):B2B-XH
- added H1, H2, H3, H4: MOUNT-HOLE3.2, holes:3,2
- added SERVO1, SERVO2: (no value), con-jst-xh (1):B3B-XH
- moved C5 8.25 mm to (35.6, 17.6)
- moved C6 8.25 mm to (36.8, 17.6)
- moved U$17 8.16 mm to (33.0, 12.9)
- moved LED 5.85 mm to (38.4, 0.90), turned to 270 degrees
- moved C4 5.39 mm to (29.1, 18.2)
- moved C1 5.39 mm to (29.1, 22.2)
- moved C2 5.39 mm to (35.6, 27.3)
- moved C3 5.39 mm to (36.8, 27.3)
- moved U$1 5.39 mm to (33.0, 25.0)
- moved AZUSA 4.00 mm to (44.4, 25.4)
- moved SW1 4.00 mm to (44.4, 34.9)
- moved SW2 4.00 mm to (34.3, 34.9)
- moved CON1 3.00 mm to (21.0, 28.0)
Connections:
- removed net PWM_SERVO: AZUSA_CON.2, SERVO.3
- new net PWM1_SERVO: AZUSA_CON1.2, SERVO1.3
- new net PWM2_SERVO: AZUSA_CON2.2, SERVO2.3
- net +6V: now also SERVO1.2, SERVO2.2; no longer SERVO.2
- net GND: now also AZUSA_CON1.1, AZUSA_CON2.1, SERVO1.1, SERVO2.1; no longer AZUSA_CON.1, SERVO.1
Routing:
- net PWM_SERVO: track 15.5 -> 0.00 mm
- net PWM2_SERVO: track 0.00 -> 14.7 mm
- net RED: track 18.1 -> 32.7 mm
- net PWM1_SERVO: track 0.00 -> 14.1 mm
- net +12V: track 11.8 -> 18.4 mm
- net BLUE: track 13.2 -> 17.2 mm
- net PVCC: track 30.0 -> 32.1 mm
- net +6V: track 43.3 -> 42.0 mm
- added copper zone on layer 16, net GND
Other:
- board size 53 x 42 mm -> 53 x 58 mm
