File: src/上昇＆摘果機構回路.brd (EAGLE design)
At the start: 97.6 x 76.1 mm, 58 parts, among them T1 2SC3325-Y,LF, X1 32.768K12.5PI/MC306, X2 RH100-24.000-18-1020-EXT-TR

Commit message: servo
Parts:
- added SERVO: 02-JST, con-jst-xh (1):B2B-XH
Connections:
- new net PWM_SERVO: SERVO.2, U$1.PB0
- net SGND: now also SERVO.1
Routing:
- net PWM_SERVO: track 0.00 -> 80.3 mm, vias 0 -> 1

Commit message: add serbo pin
Parts:
- renumbered SERVO to AZUSA_COM
Changed lines of the file:
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@@
 <attribute name="VALUE" x="71.241" y="8.632" size="1.27" layer="27" rot="R180"/>
 </element>
-<element name="SERVO" library="con-jst-xh (1)" package="B2B-XH" value="02-JST" x="90.8" y="57.8" smashed="yes" rot="R90">
+<element name="AZUSA_COM" library="con-jst-xh (1)" package="B2B-XH" value="02-JST" x="90.8" y="57.8" smashed="yes" rot="R90">
 <attribute name="NAME" x="86.99" y="56.53" size="1.27" layer="25" rot="R90"/>
 <attribute name="VALUE" x="94.61" y="56.53" size="1.27" layer="27" rot="R90"/>
@@
 <vertex x="62.7" y="7"/>
 </polygon>
-<contactref element="SERVO" pad="1"/>
+<contactref element="AZUSA_COM" pad="1"/>
 <wire x1="82.59" y1="71.59" x2="85.4" y2="73.4" width="0" layer="19" extent="1-1"/>
 <wire x1="78.8" y1="66.6" x2="82.59" y2="71.59" width="0" layer="19" extent="1-1"/>
@@
 </signal>
 <signal name="PWM_SERVO">
-<contactref element="SERVO" pad="2"/>
+<contactref element="AZUSA_COM" pad="2"/>
 <contactref element="U$1" pad="PB0"/>
 <wire x1="54.25" y1="34.4" x2="54.25" y2="32.15" width="0.2" layer="16"/>

Commit message: silk update
Parts:
- moved U$2 5.77 mm to (76.1, 43.7), turned to 90 degrees
- moved C24 4.08 mm to (71.3, 33.6), turned to 0 degrees
- moved C21 3.66 mm to (68.4, 35.7)
- moved C20 3.26 mm to (65.4, 33.6)
- moved U$8 2.73 mm to (20.9, 13.2)
- moved TWE_LEFT 2.61 mm to (13.2, 37.3)
- moved TWE_RIGHT 2.61 mm to (28.9, 37.3)
- moved R12 2.52 mm to (21.1, 9.70)
- moved C16 2.12 mm to (80.9, 33.6)
- moved R10 2.05 mm to (84.4, 46.4)
- moved C15 2.04 mm to (80.9, 35.7)
- moved C18 1.84 mm to (83.9, 33.6)
- moved C23 1.75 mm to (71.6, 36.0), turned to 0 degrees
- moved C17 1.75 mm to (83.9, 35.7)
- moved R11 1.50 mm to (84.4, 40.2)
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- renumbered JP1 to BOOT, JP8 to ST-LINK, LEFT to LEFT_U, LEFT2 to LEFT_D, RIGHT to RIGHT_U, RIGHT2 to RIGHT_D
Routing:
- net RX: track 61.0 -> 63.7 mm
- net TX: track 26.5 -> 29.0 mm
- net PGND: track 10.4 -> 12.5 mm
- net N$46: track 13.0 -> 14.8 mm
- net +5V: track 158.0 -> 159.7 mm
- net COM_LED2: track 22.6 -> 21.4 mm
- net NRST: track 48.6 -> 49.8 mm
- net N$8: track 20.0 -> 21.1 mm
- net +3V3: track 184.6 -> 185.6 mm
- net N$19: track 3.49 -> 4.29 mm
Other:
- board text added: "C5"
- board text added: "FB1"
- board text added: "T1"
- board text added: "UART_SKT"

Commit message: silk update
Parts:
- moved AZUSA_COM 0.90 mm to (90.8, 56.9)
Other:
- board text added: "RESET"
Changed lines of the file:
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@@
 <text x="44.9" y="48" size="1.27" layer="25" rot="R90">UART_SKT</text>
 <text x="67.6" y="36.5" size="0.6096" layer="25">FB1</text>
+<text x="72.3" y="40.8" size="1.27" layer="25" rot="R90">RESET</text>
 </plain>
 <attributes>
@@
 <attribute name="VALUE" x="71.241" y="8.632" size="1.27" layer="27" rot="R180"/>
 </element>
-<element name="AZUSA_COM" library="con-jst-xh (1)" package="B2B-XH" value="02-JST" x="90.8" y="57.8" smashed="yes" rot="R90">
-<attribute name="NAME" x="86.79" y="51.63" size="1.27" layer="25" rot="R90"/>
-<attribute name="VALUE" x="94.61" y="56.53" size="1.27" layer="27" rot="R90"/>
+<element name="AZUSA_COM" library="con-jst-xh (1)" package="B2B-XH" value="02-JST" x="90.8" y="56.9" smashed="yes" rot="R90">
+<attribute name="NAME" x="86.79" y="51.43" size="1.27" layer="25" rot="R90"/>
+<attribute name="VALUE" x="94.61" y="55.63" size="1.27" layer="27" rot="R90"/>
 </element>
 </elements>
@@
 <wire x1="64" y1="73.6" x2="61.01" y2="71.7" width="0" layer="19" extent="1-1"/>
 <wire x1="71.9" y1="73.5" x2="64" y2="73.6" width="0" layer="19" extent="1-1"/>
-<wire x1="90.8" y1="59.07" x2="81.6" y2="59.7" width="0" layer="19" extent="1-1"/>
+<wire x1="90.8" y1="58.17" x2="81.6" y2="59.7" width="0" layer="19" extent="1-1"/>
 <wire x1="46.6" y1="19.1" x2="43.8" y2="27.9" width="0" layer="19" extent="1-1"/>
 <wire x1="41.2" y1="15.1" x2="46.6" y2="19.1" width="0" layer="19" extent="1-1"/>
@@
 <wire x1="91.3" y1="23.3" x2="94.2" y2="26.2" width="0.2" layer="1"/>
 <wire x1="94.2" y1="26.2" x2="94.2" y2="53.3" width="0.2" layer="1"/>
-<wire x1="94.2" y1="53.3" x2="90.97" y2="56.53" width="0.2" layer="1"/>
-<wire x1="90.97" y1="56.53" x2="90.8" y2="56.53" width="0.2" layer="1"/>
+<wire x1="94.2" y1="53.3" x2="91.87" y2="55.63" width="0.2" layer="1"/>
+<wire x1="91.87" y1="55.63" x2="90.8" y2="55.63" width="0.2" layer="1"/>
 <wire x1="55.4" y1="28.6" x2="60.7" y2="23.3" width="0.2" layer="1"/>
 </signal>

Commit message: servo2
Parts:
- removed ENC4: (no value), con-jst-xh (1):B5B-XH
- added AZUSA_CON2: 02-JST, con-jst-xh (1):B2B-XH
- moved ENC3 8.70 mm to (37.0, 72.6)
- renumbered AZUSA_COM to AZUSA_CON1
Connections:
- net PWM_SERVO renamed PWM1_SERVO
- removed net EN4_A: ENC4.3, U$1.PB7
- removed net EN4_B: ENC4.5, U$1.PB6
- new net PWM2_SERVO: AZUSA_CON2.2, U$1.PB6
- net +5V: no longer ENC4.4
- net SGND: now also AZUSA_CON2.1; no longer ENC4.1
Routing:
- net EN4_A: track 41.6 -> 0.00 mm, vias 2 -> 0
- net EN4_B: track 38.6 -> 0.00 mm, vias 2 -> 0
- net EN3_B: track 26.9 -> 35.6 mm
- net EN3_A: track 31.7 -> 40.4 mm
- net +5V: track 159.7 -> 151.6 mm
- net PWM1_SERVO: track 79.9 -> 77.7 mm

Commit message: servo3
Routing:
- net PWM2_SERVO: track 0.00 -> 46.8 mm, vias 0 -> 4
- net PWM1_SERVO: track 77.7 -> 79.9 mm
- net DIR1: track 83.4 -> 82.0 mm
Changed lines of the file:
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@@
 <via x="65.9" y="47.1" extent="1-16" drill="0.35"/>
 <via x="80.6" y="42.6" extent="1-16" drill="0.35"/>
-<via x="75.9" y="54.8" extent="1-16" drill="0.35"/>
-<via x="81.5" y="61.2" extent="1-16" drill="0.35"/>
 <via x="74" y="36" extent="1-16" drill="0.35"/>
 <via x="21.1" y="58" extent="1-16" drill="0.35"/>
@@
 <contactref element="AZUSA_CON1" pad="1"/>
 <contactref element="AZUSA_CON2" pad="1"/>
+<polygon width="0.2" layer="16" pour="cutout">
+<vertex x="56" y="51.7"/>
+<vertex x="56.5" y="51.7"/>
+<vertex x="56.5" y="51.3"/>
+<vertex x="56" y="51.3"/>
+</polygon>
 </signal>
 <signal name="DIR4">
@@
 <contactref element="U$1" pad="PC5"/>
 <wire x1="54.75" y1="34.4" x2="54.7506" y2="34.3994" width="0.2" layer="16"/>
-<wire x1="54.7506" y1="34.3994" x2="54.7506" y2="32.9067625" width="0.2" layer="16"/>
 <wire x1="54.7506" y1="32.9067625" x2="56.7211625" y2="30.9362" width="0.2" layer="16"/>
 <wire x1="56.7211625" y1="30.9362" x2="75.0852" y2="30.9362" width="0.2" layer="16"/>
+<wire x1="54.7506" y1="32.9067625" x2="54.75" y2="34.4" width="0" layer="19" extent="16-16"/>
 </signal>
 <signal name="CS">
@@
 <contactref element="U$1" pad="PB6"/>
 <contactref element="AZUSA_CON2" pad="2"/>
-<wire x1="55.75" y1="45.6" x2="82.5" y2="55.43" width="0" layer="19" extent="16-16"/>
+<wire x1="55.7626" y1="45.7126" x2="55.75" y2="45.7" width="0.2" layer="16"/>
+<wire x1="55.75" y1="45.6" x2="55.75" y2="45.7" width="0.2" layer="16"/>
+<wire x1="55.7626" y1="45.7126" x2="55.7626" y2="54.78618125" width="0.2" layer="16"/>
+<wire x1="61.7" y1="56.9" x2="57.87641875" y2="56.9" width="0.2" layer="16"/>
+<wire x1="57.87641875" y1="56.9" x2="55.7626" y2="54.78618125" width="0.2" layer="16"/>
+<via x="61.7" y="56.9" extent="1-16" drill="0.35"/>
+<wire x1="61.7" y1="56.9" x2="66.9" y2="56.9" width="0.2" layer="1"/>
+<via x="66.9" y="56.9" extent="1-16" drill="0.35"/>
+<wire x1="66.9" y1="56.9" x2="75.1" y2="56.9" width="0.2" layer="16"/>
+<wire x1="75.1" y1="56.9" x2="75.9" y2="56.1" width="0.2" layer="16"/>
+<via x="75.9" y="56.1" extent="1-16" drill="0.35"/>
+<via x="81.4" y="61.3088" extent="1-16" drill="0.35"/>
+<wire x1="75.9" y1="56.1" x2="75.9" y2="59.462" width="0.2" layer="1"/>
+<wire x1="77.6988" y1="61.2608" x2="75.9" y2="59.462" width="0.2" layer="1"/>
+<wire x1="81.4" y1="61.2608" x2="77.6988" y2="61.2608" width="0.2" layer="1"/>
+<wire x1="81.4" y1="61.2608" x2="81.4" y2="61.3088" width="0.2" layer="1"/>
+<wire x1="82.5" y1="55.43" x2="81.97505" y2="55.43" width="0.2" layer="16"/>
+<wire x1="81.97505" y1="55.43" x2="81.4" y2="56.00505" width="0.2" layer="16"/>
+<wire x1="81.4" y1="61.3088" x2="81.4" y2="56.00505" width="0.2" layer="16"/>
 </signal>
 <signal name="PWM1_SERVO">
@@
 <wire x1="91.87" y1="55.63" x2="90.8" y2="55.63" width="0.2" layer="1"/>
 <wire x1="55.4" y1="28.6" x2="60.7" y2="23.3" width="0.2" layer="1"/>
-<wire x1="54.25" y1="32.15" x2="54.25" y2="34.4" width="0" layer="19" extent="16-16"/>
+<wire x1="54.25" y1="34.4" x2="54.25" y2="32.15" width="0.2" layer="16"/>
 </signal>
 </signals>

Commit message: necefunc fix
Routing:
- net DIR1: track 82.0 -> 83.4 mm
Changed lines of the file:
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@@
 <contactref element="U$1" pad="PC5"/>
 <wire x1="54.75" y1="34.4" x2="54.7506" y2="34.3994" width="0.2" layer="16"/>
-<wire x1="54.7506" y1="32.9067625" x2="56.7211625" y2="30.9362" width="0.2" layer="16"/>
 <wire x1="56.7211625" y1="30.9362" x2="75.0852" y2="30.9362" width="0.2" layer="16"/>
-<wire x1="54.7506" y1="32.9067625" x2="54.75" y2="34.4" width="0" layer="19" extent="16-16"/>
+<wire x1="54.75" y1="34.4" x2="54.75" y2="32.9073625" width="0.2" layer="16"/>
+<wire x1="54.75" y1="32.9073625" x2="56.7211625" y2="30.9362" width="0.2" layer="16"/>
 </signal>
 <signal name="CS">
