File: src/remote emergency switch.brd (EAGLE design)
At the start: 47.9 x 49.5 mm, 13 parts

Commit message: twelite
Parts:
- added H1, H2, H3: MOUNT-HOLE3.2, holes:3,2
- moved C1 0.76 mm to (14.0, 23.4)
- moved C2 0.76 mm to (14.0, 20.8)
- moved C3 0.76 mm to (11.4, 20.8)
- moved C4 0.76 mm to (11.4, 23.4)
Routing:
- net +3V3: track 83.6 -> 88.6 mm
- net EM1: track 15.8 -> 12.8 mm
- net +5V: track 17.9 -> 18.7 mm
- added copper zone on layer 16, net SGND
Other:
- outline, holes or cut-outs redrawn
