File: src/remote emergency switch.sch (EAGLE design)
At the start: 13 parts

Commit message: twelite
Parts:
- added H1, H2, H3: MOUNT-HOLE3.2, holes:MOUNT-HOLE3.2
Other:
- note added: "drill"
Changed lines of the file:
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@@
 <part name="C1" library="GRM0335C1E240GA01D" deviceset="GRM0335C1E240GA01D" device="" value="10μ"/>
 <part name="C4" library="GRM0335C1E240GA01D" deviceset="GRM0335C1E240GA01D" device="" value="22μ"/>
+<part name="H1" library="holes" library_urn="urn:adsk.eagle:library:237" deviceset="MOUNT-HOLE" device="3.2" package3d_urn="urn:adsk.eagle:package:14275/1"/>
+<part name="H2" library="holes" library_urn="urn:adsk.eagle:library:237" deviceset="MOUNT-HOLE" device="3.2" package3d_urn="urn:adsk.eagle:package:14275/1"/>
+<part name="H3" library="holes" library_urn="urn:adsk.eagle:library:237" deviceset="MOUNT-HOLE" device="3.2" package3d_urn="urn:adsk.eagle:package:14275/1"/>
 </parts>
 <sheets>
@@
 <text x="-121.92" y="-53.34" size="1.778" layer="94">センサー固有パラメーター設定を０にするとtwelite内部でプルアップする</text>
 <text x="22.86" y="5.08" size="2.54" layer="94">ミシン目（スリット）等の加工を加え、PCB製造後に切り離す</text>
+<wire x1="63.5" y1="7.62" x2="15.24" y2="7.62" width="0.1524" layer="97"/>
+<wire x1="15.24" y1="7.62" x2="15.24" y2="48.26" width="0.1524" layer="97"/>
+<wire x1="15.24" y1="48.26" x2="63.5" y2="48.26" width="0.1524" layer="97"/>
+<wire x1="63.5" y1="48.26" x2="63.5" y2="7.62" width="0.1524" layer="97"/>
+<text x="17.78" y="38.1" size="6.4516" layer="97">drill</text>
 </plain>
 <instances>
@@
 <attribute name="VALUE" x="-28.956" y="18.161" size="1.778" layer="96"/>
 </instance>
+<instance part="H1" gate="G$1" x="20.32" y="27.94" smashed="yes">
+<attribute name="NAME" x="22.352" y="28.5242" size="1.778" layer="95"/>
+<attribute name="VALUE" x="22.352" y="25.4762" size="1.778" layer="96"/>
+</instance>
+<instance part="H2" gate="G$1" x="33.02" y="27.94" smashed="yes">
+<attribute name="NAME" x="35.052" y="28.5242" size="1.778" layer="95"/>
+<attribute name="VALUE" x="35.052" y="25.4762" size="1.778" layer="96"/>
+</instance>
+<instance part="H3" gate="G$1" x="27.94" y="12.7" smashed="yes">
+<attribute name="NAME" x="29.972" y="13.2842" size="1.778" layer="95"/>
+<attribute name="VALUE" x="29.972" y="10.2362" size="1.778" layer="96"/>
+</instance>
 </instances>
