File: src/kicad/kicad 2/Mix necessary function 2/Mix necessary function.kicad_pcb (KiCad board)
At the start: 2 copper layers, 53 x 58 mm, 26 parts, among them SW1 02-JST, SW2 02-JST

Commit message: fix
Parts:
- removed Lipo＿THRU: XT90PW-M, Mix necessary function:XT90PW-M
- added D1: GS2M-LTP, Mix necessary function:GS2M-LTP, F.Cu at (139.0, 114.1)
- added LIPO＿THRU: XT90PW-M, Mix necessary function:XT90PW-M, F.Cu at (143.0, 96.2)
- added Q1: SQJA16EP-T1_GE3, Mix necessary function:SQJA16EP-T1_GE3, F.Cu at (145.0, 112.7)
- added R2: 820, Mix necessary function:CR0603, F.Cu at (137.0, 109.9)
- added R3: 10, Mix necessary function:CR0603, F.Cu at (139.0, 109.9)
- added R4: 10k, Mix necessary function:CR0603, F.Cu at (141.0, 109.9)
- added ZD1: MMBZ5248B-TP, Mix necessary function:MMBZ5248B-TP, F.Cu at (155.7, 119.0)
- moved TLP1 7.00 mm to (128.0, 113.5)
- moved C7 6.86 mm to (134.4, 109.8)
- moved R1 5.39 mm to (126.0, 113.9), turned to 90 degrees
- moved THRU 1.00 mm to (126.0, 120.0)
- moved LED 0.72 mm to (161.0, 124.5)
- moved C3 0.22 mm to (159.0, 97.7)
- moved C6 0.22 mm to (159.0, 107.4)
Connections:
- TLP1 pad VO: PVCC -> N$6
Routing:
- net N$7: track 0.00 -> 29.7 mm
- net PVCC: track 41.3 -> 69.4 mm, vias 0 -> 2
- net N$20: track 12.7 -> 33.2 mm
- net +6V: track 60.2 -> 70.8 mm
- net N$6: track 0.00 -> 6.09 mm
- net N$1: track 12.7 -> 8.13 mm
- net N$8: track 0.00 -> 4.49 mm
- net N$92: track 7.98 -> 3.81 mm
- net RED: track 32.3 -> 28.6 mm
- net PWM2_SERVO: track 14.7 -> 13.7 mm
- net +12V: track 18.4 -> 19.4 mm
- net N$118: track 3.01 -> 2.25 mm
- net BLUE: track 17.2 -> 17.8 mm
- net GND: vias 22 -> 27
Other:
- board text added: "C7"
- board text added: "D1"
- board text added: "L"
- board text added: "L:Blue R:Red"
- board text added: "R"
- board text added: "R2"
- board text added: "R3"
- board text added: "R4"
- board text added: "ZD1"
- board text removed: "L: Blue R: Red"
